Commit message: One finger gripper working in Gazebo with roscontrol

File: urdf/simple_gripper.urdf (robot description, URDF)
Before this commit: robot simple_gripper, 3 links, 2 joints
Links:
- link finger1: mass None -> 0.1; geometry collision box size=0.02 0.02 0.08; visual box size=0.02 0.02 0.08
- link finger2: mass None -> 0.1; geometry collision box size=0.02 0.02 0.08; visual box size=0.02 0.02 0.08
- link palm: mass None -> 0.1; geometry collision cylinder length=0.04 radius=0.04; visual cylinder length=0.04 radius=0.04

Commit message: Have a working model of a gripper... but contact dynamics are very nasty indeed.  Using custom shapes to try and get them to pick up cleanly, but the dumbbell still jumps around when gripped.  Have attempted tuning the material parameters and using softer control gains to achieve gentle contact... but no joy yet.

File: urdf/simple_gripper.urdf (robot description, URDF)
Before this commit: robot simple_gripper, 3 links, 2 joints
Links:
- link palm: geometry collision cylinder length=0.04 radius=0.07; visual cylinder length=0.04 radius=0.07
Joints:
- joint palm_to_finger1: origin xyz=0.03 0 0.04 -> xyz=0.05 0 0.04
- joint palm_to_finger2: limit lower=0.0 upper=0.035 effort=1000.0 velocity=0.5 -> lower=0.0 upper=0.065 effort=1000.0 velocity=0.5; origin xyz=-0.03 0 0.04 -> xyz=-0.05 0 0.04

Commit message: New attempt using gazebo_grasp_fix.  It's loaded and running - but doesn't do the trick.  Also made second finger mobile now, and added gripper utility script.

File: urdf/simple_gripper.urdf (robot description, URDF)
Before this commit: robot simple_gripper, 3 links, 2 joints
Joints:
- joint palm_to_finger1: limit (none) -> lower=0.0 upper=0.03 effort=1 velocity=0.05; origin xyz=0.05 0 0.04 -> xyz=0.05 0 0.04 rpy=0 0 3.14159265; type fixed -> prismatic
- joint palm_to_finger2: limit lower=0.0 upper=0.065 effort=1000.0 velocity=0.5 -> lower=0.0 upper=0.03 effort=1.0 velocity=0.05
