Commit message: Tuning, including trying the grasp_fix again, with bigger jaws and soft grip pads.  Still doesn't work.  Have occasionally managed some lifts with the grasp fix, but unreliably.

File: urdf/simple_gripper.urdf.xacro (robot description, xacro)
@@ -19,16 +19,20 @@
     </inertial>
   </link>
-  <link name="finger1">
+  <xacro:macro name="finger" params="suffix">
+   <link name="finger${suffix}">
     <visual>
       <geometry>
-        <box size="0.02 0.02 0.08"/>
+        <box size="0.02 0.05 0.12"/>
       </geometry>
-      <origin rpy="0 0 0" xyz="0 0 0.04"/>
+      <origin rpy="0 0 0" xyz="0 0 0.06"/>
+      <material name="fing">
+        <color rgba="0.6 0.6 0.8 1" />
+      </material>
     </visual>
     <collision>
       <geometry>
-        <box size="0.02 0.02 0.08"/>
+        <box size="0.02 0.05 0.12"/>
       </geometry>
-      <origin rpy="0 0 0" xyz="0 0 0.04"/>
+      <origin rpy="0 0 0" xyz="0 0 0.06"/>
     </collision>
     <inertial>
@@ -36,56 +40,53 @@
       <inertia ixx="0.001" ixy="0.0" ixz="0.0" iyy="0.001" iyz="0.0" izz="0.001"/>
     </inertial>
-  </link>
-  <link name="finger2">
+   </link>
+   <link name="pad${suffix}">
     <visual>
       <geometry>
-        <box size="0.02 0.02 0.08"/>
+        <box size="0.006 0.04 0.08"/>
       </geometry>
-      <origin rpy="0 0 0" xyz="0 0 0.04"/>
+      <origin rpy="0 0 0" xyz="0 0 0.02"/>
+      <material name="pad">
+        <color rgba="0.2 0.2 0.2 1" />
+      </material>
     </visual>
     <collision>
       <geometry>
-        <box size="0.02 0.02 0.08"/>
+        <box size="0.006 0.04 0.08"/>
       </geometry>
-      <origin rpy="0 0 0" xyz="0 0 0.04"/>
+      <origin rpy="0 0 0" xyz="0 0 0.02"/>
     </collision>
     <inertial>
-      <mass value="0.1"/>
+      <mass value="0.01"/>
       <inertia ixx="0.001" ixy="0.0" ixz="0.0" iyy="0.001" iyz="0.0" izz="0.001"/>
     </inertial>
-  </link>
-  <!-- make fingers soft and sticky -->
-  <!-- removing - using grasp fix instead
-  <gazebo reference="finger1">
-    <mu1 value="0.8" />
-    <mu2 value="0.8" />
+   </link>
+   <joint name="finger${suffix}_to_pad${suffix}" type="fixed">
+    <parent link="finger${suffix}"/>
+    <child link="pad${suffix}"/>
+    <origin xyz="0.013 0 0.06"/>
+   </joint>
+   <!-- make the pad squishy -->
+   <gazebo reference="pad${suffix}">
+    <mu1 value="10.0" />
+    <mu2 value="10.0" />
     <kp  value="10000000" />
-  </gazebo>
-  <gazebo reference="finger2">
-    <mu1 value="0.8" />
-    <mu2 value="0.8" />
-    <kp  value="10000000" />
-  </gazebo>
-  -->
-  <!-- one finger is fixed -->
-  <!--
-  <joint name="palm_to_finger1" type="fixed">
-    <parent link="palm"/>
-    <child link="finger1"/>
-    <origin xyz="0.05 0 0.04"/>
-  </joint>
-  -->
+   </gazebo>
+  </xacro:macro>
+  <!-- make two fingers -->
+  <xacro:finger suffix="1" />
+  <xacro:finger suffix="2" />
   <!-- fingers can slide -->
   <joint name="palm_to_finger1" type="prismatic">
     <parent link="palm"/>
     <child link="finger1"/>
-    <limit effort="1" lower="0.0" upper="0.03" velocity="0.05"/>
-    <origin xyz="0.05 0 0.04" rpy="0 0 3.14159265"/>
+    <limit effort="100.0" lower="0.0" upper="0.045" velocity="0.05"/>
+    <origin xyz="0.06 0 0.04" rpy="0 0 3.14159265"/>
   </joint>
   <joint name="palm_to_finger2" type="prismatic">
     <parent link="palm"/>
     <child link="finger2"/>
-    <limit effort="1.0" lower="0.0" upper="0.03" velocity="0.05"/>
-    <origin xyz="-0.05 0 0.04"/>
+    <limit effort="100.0" lower="0.0" upper="0.045" velocity="0.05"/>
+    <origin xyz="-0.06 0 0.04"/>
   </joint>
   <transmission name="finger1_trans">
@@ -114,7 +115,7 @@
         <arm>
            <arm_name>arm</arm_name>
-           <palm_link> wrist_3_link  </palm_link>
-           <gripper_link> finger1 </gripper_link>
-           <gripper_link> finger2 </gripper_link>
+           <palm_link>wrist_3_link</palm_link>
+           <gripper_link>finger1</gripper_link>
+           <gripper_link>finger2</gripper_link>
         </arm>
         <forces_angle_tolerance>100</forces_angle_tolerance>
@@ -122,5 +123,5 @@
         <grip_count_threshold>4</grip_count_threshold>
         <max_grip_count>8</max_grip_count>
-        <release_tolerance>0.005</release_tolerance>
+        <release_tolerance>0.01</release_tolerance>
         <disable_collisions_on_attach>false</disable_collisions_on_attach>
         <contact_topic>__default_topic__</contact_topic>

Commit message: Gripper narrower in case need to pick up from ground.

File: urdf/simple_gripper.urdf.xacro (robot description, xacro)
@@ -4,5 +4,5 @@
     <visual>
       <geometry>
-        <cylinder length="0.04" radius="0.1"/>
+        <box size="0.2 0.1 0.04" />
       </geometry>
       <origin rpy="0 0 0" xyz="0 0 0.02"/>
@@ -10,5 +10,5 @@
     <collision>
       <geometry>
-        <cylinder length="0.04" radius="0.07"/>
+        <box size="0.2 0.1 0.04" />
       </geometry>
       <origin rpy="0 0 0" xyz="0 0 0.02"/>

Commit message: Working manually.  Can pick up and drop off using manual scripts and looking.

File: urdf/simple_gripper.urdf.xacro (robot description, xacro)
@@ -53,5 +53,5 @@
     <collision>
       <geometry>
-        <box size="0.006 0.04 0.08"/>
+        <box size="0.020 0.04 0.08"/>
       </geometry>
       <origin rpy="0 0 0" xyz="0 0 0.02"/>
@@ -65,5 +65,5 @@
     <parent link="finger${suffix}"/>
     <child link="pad${suffix}"/>
-    <origin xyz="0.013 0 0.06"/>
+    <origin xyz="0.013 0 0.06" rpy="0 0.1 0"/>
    </joint>
    <!-- make the pad squishy -->
