Commit message: ros control loaded and can move the arm.  Problems with showing the hand.  Don't seem to be able to move it at all yet.

File: urdf/farscope_robot.urdf.xacro (robot description, xacro)
@@ -11,5 +11,5 @@
   <xacro:include filename="$(find ur_description)/urdf/ur10.urdf.xacro" />
   <!-- make the arm -->
-  <xacro:ur10_robot prefix="ur10_" joint_limited="true"
+  <xacro:ur10_robot prefix="" joint_limited="true"
     shoulder_pan_lower_limit="${-pi}" shoulder_pan_upper_limit="${pi}"
     shoulder_lift_lower_limit="${-pi}" shoulder_lift_upper_limit="${pi}"
@@ -22,5 +22,5 @@
   <!-- fix the gripper to the arm -->
   <joint name="gripper_base_joint" type="fixed">
-    <parent link="ur10_tool0" />
+    <parent link="tool0" />
     <child link = "robotiq_arg2f_base_link" />
     <origin xyz="0.0 0.0 0.0" rpy="0.0 0.0 0.0" />
@@ -30,5 +30,5 @@
   <joint name="arm_base_joint" type="fixed">
     <parent link="world" />
-    <child link = "ur10_base_link" />
+    <child link = "base_link" />
     <origin xyz="0.0 0.0 0.0" rpy="0.0 0.0 0.0" />
   </joint>

Commit message: Basic visualization of 1-DOF gripper

File: urdf/farscope_robot.urdf.xacro (robot description, xacro)
@@ -2,6 +2,5 @@
 <robot name="farscope_robot" xmlns:xacro="http://ros.org/wiki/xacro">
   <!-- gripper -->
-  <xacro:include filename="$(find robotiq_2f_85_gripper_visualization)/urdf/robotiq_arg2f_85_model_macro.xacro" />
-  <xacro:robotiq_arg2f_85 prefix=""/>
+  <xacro:include filename="$(find farscope_group_proj)/urdf/simple_gripper.urdf" />
   <!-- arm (copied from ur_description/urdf/ur10_joint_limited.urdf.xacro) -->
   <xacro:arg name="transmission_hw_interface" default="hardware_interface/PositionJointInterface"/>
@@ -23,5 +22,5 @@
   <joint name="gripper_base_joint" type="fixed">
     <parent link="tool0" />
-    <child link = "robotiq_arg2f_base_link" />
+    <child link = "palm" />
     <origin xyz="0.0 0.0 0.0" rpy="0.0 0.0 0.0" />
   </joint>

Commit message: URDF now integrates MPO700 base and cabinet.  Note new dependency on neo_simulation (but unmodified - no need for fork).  TODO get integrated robot in Gazebo.

File: urdf/farscope_robot.urdf.xacro (robot description, xacro)
@@ -1,7 +1,10 @@
 <?xml version="1.0"?>
 <robot name="farscope_robot" xmlns:xacro="http://ros.org/wiki/xacro">
-  <!-- gripper -->
+  <!-- ************************************ -->
+  <!-- ****** gripper ****** -->
   <xacro:include filename="$(find farscope_group_proj)/urdf/simple_gripper.urdf.xacro" />
-  <!-- arm (copied from ur_description/urdf/ur10_joint_limited.urdf.xacro) -->
+  <!-- ************************************ -->
+  <!-- ****** arm stuff ****** -->
+  <!-- copied from ur_description/urdf/ur10_joint_limited.urdf.xacro -->
   <xacro:arg name="transmission_hw_interface" default="hardware_interface/PositionJointInterface"/>
   <!-- common stuff -->
@@ -10,5 +13,5 @@
   <xacro:include filename="$(find ur_description)/urdf/ur10.urdf.xacro" />
   <!-- make the arm -->
-  <xacro:ur10_robot prefix="" joint_limited="true"
+  <xacro:ur10_robot prefix="arm_" joint_limited="true"
     shoulder_pan_lower_limit="${-pi}" shoulder_pan_upper_limit="${pi}"
     shoulder_lift_lower_limit="${-pi}" shoulder_lift_upper_limit="${pi}"
@@ -19,16 +22,70 @@
     transmission_hw_interface="$(arg transmission_hw_interface)"
 />
+  <!-- ************************************ -->
+  <!-- ****** build the mobile base ****** -->
+  <!-- adapting from neo_simulation:mmo700.urdf.xacro -->
+  <!--mmo700 common stuff -->
+  <xacro:include filename="$(find neo_simulation)/robots/mmo_700/urdf/xacros/common.gazebo.xacro" />
+  <!-- CABINET -->
+  <xacro:include filename="$(find neo_simulation)/robots/mmo_700/urdf/xacros/cabinet.xacro" />
+  <!-- Body -->
+  <xacro:include filename="$(find neo_simulation)/robots/mmo_700/urdf/xacros/mpo_700_body.xacro" />
+  <!-- SENSORS -->
+  <!-- Sick-S300 -->
+  <!-- <xacro:include filename="$(find neo_simulation)/robots/mmo_700/xacros/sick_S300.xacro" /> -->
+  <!--Sick Micro-scan  -->
+  <xacro:include filename="$(find neo_simulation)/robots/mmo_700/urdf/xacros/micro_scan.xacro" />
+  <!-- Gazebo -->
+  <xacro:include filename="$(find neo_simulation)/robots/mmo_700/urdf/xacros/mpo_700_gazebo.xacro" />
+  <!-- Head -->
+  <xacro:include filename="$(find neo_simulation)/robots/mmo_700/urdf/xacros/mpo_700_caster.xacro" />
+  <!-- Wheel -->
+  <xacro:include filename="$(find neo_simulation)/robots/mmo_700/urdf/xacros/mpo_700_wheel.xacro" />
+  <!-- Base Macro-->
+  <xacro:mpo_700_base name="base_link">
+  </xacro:mpo_700_base>
+<xacro:mpo_700_caster_0 name="mpo_700_caster_front_left" parent="base_link">
+    <origin xyz="0.24 0.18 0.27" rpy="3.14 0 -1.57" />
+  </xacro:mpo_700_caster_0>
+<!-- Casters -->
+<xacro:mpo_700_caster_1 name="mpo_700_caster_front_right" parent="base_link">
+    <origin xyz="0.24 -0.18 0.27" rpy="3.14 0 1.57" />
+  </xacro:mpo_700_caster_1>
+<xacro:mpo_700_caster_2 name="mpo_700_caster_back_left" parent="base_link">
+    <origin xyz="-0.24 0.18 0.27" rpy="3.14 0 -1.57" />
+  </xacro:mpo_700_caster_2>
+<xacro:mpo_700_caster_3 name="mpo_700_caster_back_right" parent="base_link">
+    <origin xyz="-0.24 -0.18 0.27" rpy="3.14 0 1.57" />
+  </xacro:mpo_700_caster_3>
+<!-- wheels -->
+<xacro:mpo_700_wheel name="mpo_700_wheel_front_left" parent="mpo_700_caster_front_left_link">
+    <origin xyz="-0.05 0. 0.18" rpy="0 0 0" />
+  </xacro:mpo_700_wheel>
+<xacro:mpo_700_wheel name="mpo_700_wheel_front_right" parent="mpo_700_caster_front_right_link">
+    <origin xyz="-0.05 0. 0.18" rpy="0 0 0" />
+  </xacro:mpo_700_wheel>
+<xacro:mpo_700_wheel name="mpo_700_wheel_back_left" parent="mpo_700_caster_back_left_link">
+    <origin xyz="-0.05 0. 0.18" rpy="0 0 0" />
+  </xacro:mpo_700_wheel>
+<xacro:mpo_700_wheel name="mpo_700_wheel_back_right" parent="mpo_700_caster_back_right_link">
+    <origin xyz="-0.05 0. 0.18" rpy="0 0 0" />
+  </xacro:mpo_700_wheel>
+<!--cabinet-->
+  <xacro:mmo_700_cabinet name="cabinet" parent="base_link">
+  	<origin xyz="0.072 0 0.35" rpy="0 0 0" />
+  </xacro:mmo_700_cabinet>
+  <!-- ************************************ -->
+  <!-- ****** integration ****** -->
   <!-- fix the gripper to the arm -->
   <joint name="gripper_base_joint" type="fixed">
-    <parent link="tool0" />
+    <parent link="arm_tool0" />
     <child link = "palm" />
     <origin xyz="0.0 0.0 0.0" rpy="0.0 0.0 0.0" />
   </joint>
-  <!-- fix the robot to the world -->
-  <link name="world" />
+  <!-- fix the arm to the cabinet -->
   <joint name="arm_base_joint" type="fixed">
-    <parent link="world" />
-    <child link = "base_link" />
-    <origin xyz="0.0 0.0 0.0" rpy="0.0 0.0 0.0" />
+    <parent link="cabinet_link" />
+    <child link = "arm_base_link" />
+    <origin xyz="0.133 0.0 0.416" rpy="0.0 0.0 0.0" />
   </joint>
 </robot>

Commit message: Robot now mobile in Gazebo.

File: urdf/farscope_robot.urdf.xacro (robot description, xacro)
@@ -13,5 +13,5 @@
   <xacro:include filename="$(find ur_description)/urdf/ur10.urdf.xacro" />
   <!-- make the arm -->
-  <xacro:ur10_robot prefix="arm_" joint_limited="true"
+  <xacro:ur10_robot prefix="" joint_limited="true"
     shoulder_pan_lower_limit="${-pi}" shoulder_pan_upper_limit="${pi}"
     shoulder_lift_lower_limit="${-pi}" shoulder_lift_upper_limit="${pi}"
@@ -25,6 +25,6 @@
   <!-- ****** build the mobile base ****** -->
   <!-- adapting from neo_simulation:mmo700.urdf.xacro -->
-  <!--mmo700 common stuff -->
-  <xacro:include filename="$(find neo_simulation)/robots/mmo_700/urdf/xacros/common.gazebo.xacro" />
+  <!--mmo700 common stuff SKIPPED because it reloads controllers and grasp fix-->
+  <!-- <xacro:include filename="$(find neo_simulation)/robots/mmo_700/urdf/xacros/common.gazebo.xacro" /> -->
   <!-- CABINET -->
   <xacro:include filename="$(find neo_simulation)/robots/mmo_700/urdf/xacros/cabinet.xacro" />
@@ -43,17 +43,31 @@
   <xacro:include filename="$(find neo_simulation)/robots/mmo_700/urdf/xacros/mpo_700_wheel.xacro" />
   <!-- Base Macro-->
-  <xacro:mpo_700_base name="base_link">
+  <xacro:mpo_700_base name="mpo_700_base_link">
   </xacro:mpo_700_base>
-<xacro:mpo_700_caster_0 name="mpo_700_caster_front_left" parent="base_link">
+  <!-- copied from mpo_700_gazebo.xacro -->
+   <gazebo reference="mpo_700_base_link">
+    <gravity>true</gravity>
+    <self_collide>false</self_collide>
+  </gazebo>
+<gazebo>
+    <plugin name="mpo_700_controller" filename="libgazebo_ros_planar_move.so">
+        <commandTopic>cmd_vel</commandTopic>
+        <odometryTopic>odom</odometryTopic>
+        <odometryFrame>odom</odometryFrame>
+        <odometryRate>20.0</odometryRate>
+        <robotBaseFrame>mpo_700_base_link</robotBaseFrame>
+    </plugin>
+</gazebo>
+<xacro:mpo_700_caster_0 name="mpo_700_caster_front_left" parent="mpo_700_base_link">
     <origin xyz="0.24 0.18 0.27" rpy="3.14 0 -1.57" />
   </xacro:mpo_700_caster_0>
 <!-- Casters -->
-<xacro:mpo_700_caster_1 name="mpo_700_caster_front_right" parent="base_link">
+<xacro:mpo_700_caster_1 name="mpo_700_caster_front_right" parent="mpo_700_base_link">
     <origin xyz="0.24 -0.18 0.27" rpy="3.14 0 1.57" />
   </xacro:mpo_700_caster_1>
-<xacro:mpo_700_caster_2 name="mpo_700_caster_back_left" parent="base_link">
+<xacro:mpo_700_caster_2 name="mpo_700_caster_back_left" parent="mpo_700_base_link">
     <origin xyz="-0.24 0.18 0.27" rpy="3.14 0 -1.57" />
   </xacro:mpo_700_caster_2>
-<xacro:mpo_700_caster_3 name="mpo_700_caster_back_right" parent="base_link">
+<xacro:mpo_700_caster_3 name="mpo_700_caster_back_right" parent="mpo_700_base_link">
     <origin xyz="-0.24 -0.18 0.27" rpy="3.14 0 1.57" />
   </xacro:mpo_700_caster_3>
@@ -72,5 +86,5 @@
   </xacro:mpo_700_wheel>
 <!--cabinet-->
-  <xacro:mmo_700_cabinet name="cabinet" parent="base_link">
+  <xacro:mmo_700_cabinet name="cabinet" parent="mpo_700_base_link">
   	<origin xyz="0.072 0 0.35" rpy="0 0 0" />
   </xacro:mmo_700_cabinet>
@@ -78,13 +92,13 @@
   <!-- ****** integration ****** -->
   <!-- fix the gripper to the arm -->
-  <joint name="gripper_base_joint" type="fixed">
-    <parent link="arm_tool0" />
+  <joint name="gripper_to_arm" type="fixed">
+    <parent link="tool0" />
     <child link = "palm" />
     <origin xyz="0.0 0.0 0.0" rpy="0.0 0.0 0.0" />
   </joint>
   <!-- fix the arm to the cabinet -->
-  <joint name="arm_base_joint" type="fixed">
+  <joint name="arm_to_cabinet" type="fixed">
     <parent link="cabinet_link" />
-    <child link = "arm_base_link" />
+    <child link = "base_link" />
     <origin xyz="0.133 0.0 0.416" rpy="0.0 0.0 0.0" />
   </joint>

Commit message: Wider gripper reach for better dropping.

File: urdf/farscope_robot.urdf.xacro (robot description, xacro)
@@ -37,5 +37,19 @@
   <xacro:include filename="$(find neo_simulation)/robots/mmo_700/urdf/xacros/micro_scan.xacro" />
   <!-- Gazebo -->
-  <xacro:include filename="$(find neo_simulation)/robots/mmo_700/urdf/xacros/mpo_700_gazebo.xacro" />
+  <!-- <xacro:include filename="$(find neo_simulation)/robots/mmo_700/urdf/xacros/mpo_700_gazebo.xacro" /> -->
+  <!-- copied from mpo_700_gazebo.xacro -->
+  <gazebo reference="mpo_700_base_link">
+    <gravity>true</gravity>
+    <self_collide>false</self_collide>
+  </gazebo>
+  <gazebo>
+    <plugin name="mpo_700_controller" filename="libgazebo_ros_planar_move.so">
+        <commandTopic>cmd_vel</commandTopic>
+        <odometryTopic>odom</odometryTopic>
+        <odometryFrame>odom</odometryFrame>
+        <odometryRate>20.0</odometryRate>
+        <robotBaseFrame>mpo_700_base_link</robotBaseFrame>
+    </plugin>
+  </gazebo>
   <!-- Head -->
   <xacro:include filename="$(find neo_simulation)/robots/mmo_700/urdf/xacros/mpo_700_caster.xacro" />
@@ -45,45 +59,31 @@
   <xacro:mpo_700_base name="mpo_700_base_link">
   </xacro:mpo_700_base>
-  <!-- copied from mpo_700_gazebo.xacro -->
-   <gazebo reference="mpo_700_base_link">
-    <gravity>true</gravity>
-    <self_collide>false</self_collide>
-  </gazebo>
-<gazebo>
-    <plugin name="mpo_700_controller" filename="libgazebo_ros_planar_move.so">
-        <commandTopic>cmd_vel</commandTopic>
-        <odometryTopic>odom</odometryTopic>
-        <odometryFrame>odom</odometryFrame>
-        <odometryRate>20.0</odometryRate>
-        <robotBaseFrame>mpo_700_base_link</robotBaseFrame>
-    </plugin>
-</gazebo>
-<xacro:mpo_700_caster_0 name="mpo_700_caster_front_left" parent="mpo_700_base_link">
+  <!-- Casters -->
+  <xacro:mpo_700_caster_0 name="mpo_700_caster_front_left" parent="mpo_700_base_link">
     <origin xyz="0.24 0.18 0.27" rpy="3.14 0 -1.57" />
   </xacro:mpo_700_caster_0>
-<!-- Casters -->
-<xacro:mpo_700_caster_1 name="mpo_700_caster_front_right" parent="mpo_700_base_link">
+  <xacro:mpo_700_caster_1 name="mpo_700_caster_front_right" parent="mpo_700_base_link">
     <origin xyz="0.24 -0.18 0.27" rpy="3.14 0 1.57" />
   </xacro:mpo_700_caster_1>
-<xacro:mpo_700_caster_2 name="mpo_700_caster_back_left" parent="mpo_700_base_link">
+  <xacro:mpo_700_caster_2 name="mpo_700_caster_back_left" parent="mpo_700_base_link">
     <origin xyz="-0.24 0.18 0.27" rpy="3.14 0 -1.57" />
   </xacro:mpo_700_caster_2>
-<xacro:mpo_700_caster_3 name="mpo_700_caster_back_right" parent="mpo_700_base_link">
+  <xacro:mpo_700_caster_3 name="mpo_700_caster_back_right" parent="mpo_700_base_link">
     <origin xyz="-0.24 -0.18 0.27" rpy="3.14 0 1.57" />
   </xacro:mpo_700_caster_3>
-<!-- wheels -->
-<xacro:mpo_700_wheel name="mpo_700_wheel_front_left" parent="mpo_700_caster_front_left_link">
+  <!-- wheels -->
+  <xacro:mpo_700_wheel name="mpo_700_wheel_front_left" parent="mpo_700_caster_front_left_link">
     <origin xyz="-0.05 0. 0.18" rpy="0 0 0" />
   </xacro:mpo_700_wheel>
-<xacro:mpo_700_wheel name="mpo_700_wheel_front_right" parent="mpo_700_caster_front_right_link">
+  <xacro:mpo_700_wheel name="mpo_700_wheel_front_right" parent="mpo_700_caster_front_right_link">
     <origin xyz="-0.05 0. 0.18" rpy="0 0 0" />
   </xacro:mpo_700_wheel>
-<xacro:mpo_700_wheel name="mpo_700_wheel_back_left" parent="mpo_700_caster_back_left_link">
+  <xacro:mpo_700_wheel name="mpo_700_wheel_back_left" parent="mpo_700_caster_back_left_link">
     <origin xyz="-0.05 0. 0.18" rpy="0 0 0" />
   </xacro:mpo_700_wheel>
-<xacro:mpo_700_wheel name="mpo_700_wheel_back_right" parent="mpo_700_caster_back_right_link">
+  <xacro:mpo_700_wheel name="mpo_700_wheel_back_right" parent="mpo_700_caster_back_right_link">
     <origin xyz="-0.05 0. 0.18" rpy="0 0 0" />
   </xacro:mpo_700_wheel>
-<!--cabinet-->
+  <!--cabinet-->
   <xacro:mmo_700_cabinet name="cabinet" parent="mpo_700_base_link">
   	<origin xyz="0.072 0 0.35" rpy="0 0 0" />

File: urdf/simple_gripper.urdf.xacro (robot description, xacro)
@@ -4,5 +4,5 @@
     <visual>
       <geometry>
-        <cylinder length="0.04" radius="0.07"/>
+        <cylinder length="0.04" radius="0.1"/>
       </geometry>
       <origin rpy="0 0 0" xyz="0 0 0.02"/>
@@ -81,5 +81,5 @@
     <parent link="palm"/>
     <child link="finger1"/>
-    <limit effort="100.0" lower="0.0" upper="0.045" velocity="0.05"/>
+    <limit effort="100.0" lower="-0.03" upper="0.045" velocity="0.05"/>
     <origin xyz="0.06 0 0.04" rpy="0 0 3.14159265"/>
   </joint>
@@ -87,5 +87,5 @@
     <parent link="palm"/>
     <child link="finger2"/>
-    <limit effort="100.0" lower="0.0" upper="0.045" velocity="0.05"/>
+    <limit effort="100.0" lower="-0.03" upper="0.045" velocity="0.05"/>
     <origin xyz="-0.06 0 0.04"/>
   </joint>

Commit message: LIDAR working now.  Use RVIZ to see it.

File: urdf/farscope_robot.urdf.xacro (robot description, xacro)
@@ -89,4 +89,49 @@
   	<origin xyz="0.072 0 0.35" rpy="0 0 0" />
   </xacro:mmo_700_cabinet>
+  <!-- LIDAR -->
+  <xacro:sick_laser_v0 name="lidar_1" parent="mpo_700_base_link" ros_topic="lidar_1/scan_filtered">
+  <origin xyz="0.360 0 0.181" rpy="3.14 0 0" />
+  </xacro:sick_laser_v0>
+  <!-- Lidar sensors -->
+  <gazebo reference="lidar_1_link">
+      <sensor type="ray" name="lidar_1_sensor">
+          <pose>0 0 0 0 0 0</pose>
+          <visualize>false</visualize>
+          <update_rate>40</update_rate>
+          <ray>
+            <scan>
+              <horizontal>
+                <samples>720</samples>
+                <resolution>1</resolution>
+                <min_angle>-1.48</min_angle>
+                <max_angle>1.48</max_angle>
+              </horizontal>
+            </scan>
+            <range>
+              <min>0.10</min>
+              <max>30.0</max>
+              <resolution>0.05</resolution>
+            </range>
+            <noise>
+              <type>gaussian</type>
+              <!-- Noise parameters based on published spec for Hokuyo laser
+                   achieving "+-30mm" accuracy at range < 10m.  A mean of 0.0m and
+                   stddev of 0.01m will put 99.7% of samples within 0.03m of the true
+                   reading. -->
+              <mean>0.0</mean>
+              <stddev>0.01</stddev>
+            </noise>
+          </ray>
+          <plugin name="lidar_1" filename="libgazebo_ros_laser.so">
+            <topicName>lidar_1/scan_filtered</topicName>
+            <frameName>lidar_1_link</frameName>
+          </plugin>
+        </sensor>
+  </gazebo>
+  <!--Camera  -->
+  <!--><xacro:camera name="camera" parent="base_link">
+    <origin xyz="0 0 0.38" rpy="0 0 0" />
+  </xacro:camera>
+  <-->
   <!-- ************************************ -->
   <!-- ****** integration ****** -->

Commit message: Camera added and working.  In the wrong place and direction though - make optional and customizable?

File: urdf/farscope_robot.urdf.xacro (robot description, xacro)
@@ -129,9 +129,48 @@
         </sensor>
   </gazebo>
+  <gazebo reference="camera_link">
+    <sensor type="camera" name="camera1">
+      <update_rate>30.0</update_rate>
+      <camera name="head">
+        <horizontal_fov>1.3962634</horizontal_fov>
+        <image>
+          <width>800</width>
+          <height>800</height>
+          <format>R8G8B8</format>
+        </image>
+        <clip>
+          <near>0.02</near>
+          <far>300</far>
+        </clip>
+        <noise>
+          <type>gaussian</type>
+          <!-- Noise is sampled independently per pixel on each frame.
+               That pixel's noise value is added to each of its color
+               channels, which at that point lie in the range [0,1]. -->
+          <mean>0.0</mean>
+          <stddev>0.007</stddev>
+        </noise>
+      </camera>
+      <plugin name="camera_controller" filename="libgazebo_ros_camera.so">
+        <alwaysOn>true</alwaysOn>
+        <updateRate>0.0</updateRate>
+        <cameraName>camera1</cameraName>
+        <imageTopicName>image_raw</imageTopicName>
+        <cameraInfoTopicName>camera_info</cameraInfoTopicName>
+        <frameName>camera_link</frameName>
+        <hackBaseline>0.07</hackBaseline>
+        <distortionK1>0.0</distortionK1>
+        <distortionK2>0.0</distortionK2>
+        <distortionK3>0.0</distortionK3>
+        <distortionT1>0.0</distortionT1>
+        <distortionT2>0.0</distortionT2>
+      </plugin>
+    </sensor>
+  </gazebo>
   <!--Camera  -->
-  <!--><xacro:camera name="camera" parent="base_link">
-    <origin xyz="0 0 0.38" rpy="0 0 0" />
+  <xacro:include filename="$(find neo_simulation)/robots/mmo_700/urdf/xacros/camera.xacro" />
+  <xacro:camera name="camera" parent="forearm_link" >
+    <origin xyz="0 -0.08 0.38" rpy="0 0 0" />
   </xacro:camera>
-  <-->
   <!-- ************************************ -->
   <!-- ****** integration ****** -->

Commit message: Fixed interia warning with dummy link at base.  Not sure yet if it's fixed the MPO rolling behaviour.  Also now spawns world with shelf and pallet for contest.

File: urdf/farscope_robot.urdf.xacro (robot description, xacro)
@@ -187,3 +187,9 @@
     <origin xyz="0.133 0.0 0.416" rpy="0.0 0.0 0.0" />
   </joint>
+  <!-- dummy link to avoid inertia warning -->
+  <link name="dummy_base" />
+  <joint name="dummy_joint" type="fixed">
+    <parent link="dummy_base" />
+    <child link = "mpo_700_base_link" />
+  </joint>
 </robot>

Commit message: Improved initial camera view.  Fixed colours of gripper and target.

File: urdf/farscope_robot.urdf.xacro (robot description, xacro)
@@ -173,5 +173,5 @@
   <xacro:include filename="$(find neo_simulation)/robots/mmo_700/urdf/xacros/camera.xacro" />
   <xacro:camera name="camera" parent="forearm_link" >
-    <origin xyz="0 -0.08 0.38" rpy="0 0 0" />
+    <origin xyz="0 -0.08 0.38" rpy="0 -1.5706 0" />
   </xacro:camera>
   <!-- ************************************ -->

File: urdf/simple_gripper.urdf.xacro (robot description, xacro)
@@ -7,4 +7,7 @@
       </geometry>
       <origin rpy="0 0 0" xyz="0 0 0.02"/>
+      <material name="palm">
+        <color rgba="1 0.5 0 1" />
+      </material>
     </visual>
     <collision>
@@ -19,4 +22,7 @@
     </inertial>
   </link>
+  <gazebo reference="palm">
+    <material>Gazebo/Orange</material>
+  </gazebo>
   <xacro:macro name="finger" params="suffix">
    <link name="finger${suffix}">
@@ -27,5 +33,5 @@
       <origin rpy="0 0 0" xyz="0 0 0.06"/>
       <material name="fing">
-        <color rgba="0.6 0.6 0.8 1" />
+        <color rgba="1 0.5 0 1" />
       </material>
     </visual>
@@ -41,8 +47,11 @@
     </inertial>
    </link>
+   <gazebo reference="finger${suffix}">
+     <material>Gazebo/Orange</material>
+   </gazebo>
    <link name="pad${suffix}">
     <visual>
       <geometry>
-        <box size="0.006 0.04 0.08"/>
+        <box size="0.02 0.04 0.08"/>
       </geometry>
       <origin rpy="0 0 0" xyz="0 0 0.02"/>
@@ -53,5 +62,5 @@
     <collision>
       <geometry>
-        <box size="0.020 0.04 0.08"/>
+        <box size="0.02 0.04 0.08"/>
       </geometry>
       <origin rpy="0 0 0" xyz="0 0 0.02"/>
@@ -62,4 +71,7 @@
     </inertial>
    </link>
+   <gazebo reference="pad${suffix}">
+     <material>Gazebo/Grey</material>
+   </gazebo>
    <joint name="finger${suffix}_to_pad${suffix}" type="fixed">
     <parent link="finger${suffix}"/>

Commit message: Improved handling and appearance of camera. TODO sort out Gazebo for it as well.

File: urdf/farscope_robot.urdf.xacro (robot description, xacro)
@@ -171,8 +171,5 @@
   </gazebo>
   <!--Camera  -->
-  <xacro:include filename="$(find neo_simulation)/robots/mmo_700/urdf/xacros/camera.xacro" />
-  <xacro:camera name="camera" parent="forearm_link" >
-    <origin xyz="0 -0.08 0.38" rpy="0 -1.5706 0" />
-  </xacro:camera>
+  <xacro:include filename="$(find farscope_group_proj)/urdf/simple_camera.urdf.xacro" />
   <!-- ************************************ -->
   <!-- ****** integration ****** -->
@@ -195,3 +192,8 @@
     <child link = "mpo_700_base_link" />
   </joint>
+  <joint name="camera_to_robot" type="fixed">
+    <parent link="forearm_link" />
+    <child link = "camera_link" />
+    <origin xyz="0 -0.08 0.38" rpy="0 -1.5706 0" />
+  </joint>
 </robot>
