Commit message: Camera looks better in Gazebo and frames aligned correctly.

File: urdf/farscope_robot.urdf.xacro (robot description, xacro)
@@ -131,5 +131,5 @@
   <!-- camera gazebo stuff -->
   <!-- comes first as "include" defines a camera macro, clashing in xacro with the camera block of the following -->
-  <gazebo reference="camera_link">
+  <gazebo reference="camera_lens">
     <sensor type="camera" name="camera1">
       <update_rate>30.0</update_rate>
@@ -160,5 +160,5 @@
         <imageTopicName>image_raw</imageTopicName>
         <cameraInfoTopicName>camera_info</cameraInfoTopicName>
-        <frameName>camera_link</frameName>
+        <frameName>camera_lens</frameName>
         <hackBaseline>0.07</hackBaseline>
         <distortionK1>0.0</distortionK1>

File: urdf/simple_camera.urdf.xacro (robot description, xacro)
@@ -24,7 +24,10 @@
     </inertial>
   </link>
+  <gazebo reference="camera_link">
+    <material>Gazebo/Turquoise</material>
+  </gazebo>
   <link name="camera_lens">
     <collision>
-      <origin xyz="0 0 0" rpy="0 0 0"/>
+      <origin xyz="0.0 0.0 0.0" rpy="0.0 1.5706 0.0" />
       <geometry>
         <cylinder radius="0.02" length="0.01" />
@@ -32,4 +35,5 @@
     </collision>
     <visual>
+      <origin xyz="0.0 0.0 0.0" rpy="0.0 1.5706 0.0" />
       <origin xyz="0 0 0" rpy="0 0 0"/>
       <geometry>
@@ -42,12 +46,16 @@
     <inertial>
       <mass value="1e-5" />
+      <origin xyz="0.0 0.0 0.0" rpy="0.0 1.5706 0.0" />
       <origin xyz="0 0 0" rpy="0 0 0"/>
       <inertia ixx="1e-6" ixy="0" ixz="0" iyy="1e-6" iyz="0" izz="1e-6" />
     </inertial>
   </link>
+  <gazebo reference="camera_lens">
+    <material>Gazebo/DarkGrey</material>
+  </gazebo>
   <joint name="camera_to_lens" type="fixed">
     <parent link="camera_link" />
     <child link = "camera_lens" />
-    <origin xyz="0.025 0.0 0.0" rpy="0.0 1.5706 0.0" />
+    <origin xyz="0.03 0 0" rpy="0 0 0"/>
   </joint>
 </robot>

Commit message: Camera mount is now variable by launch argument.  See farscope_robot_cam2_gazebo.launch for details.

File: urdf/farscope_robot.urdf.xacro (robot description, xacro)
@@ -7,5 +7,4 @@
   <!-- ****** arm stuff ****** -->
   <!-- copied from ur_description/urdf/ur10_joint_limited.urdf.xacro -->
-  <xacro:arg name="transmission_hw_interface" default="hardware_interface/PositionJointInterface"/>
   <!-- common stuff -->
   <xacro:include filename="$(find ur_description)/urdf/common.gazebo.xacro" />
@@ -20,5 +19,5 @@
     wrist_2_lower_limit="${-pi}" wrist_2_upper_limit="${pi}"
     wrist_3_lower_limit="${-pi}" wrist_3_upper_limit="${pi}"
-    transmission_hw_interface="$(arg transmission_hw_interface)"
+    transmission_hw_interface="hardware_interface/PositionJointInterface"
 />
   <!-- ************************************ -->
@@ -129,46 +128,6 @@
         </sensor>
   </gazebo>
-  <!-- camera gazebo stuff -->
-  <!-- comes first as "include" defines a camera macro, clashing in xacro with the camera block of the following -->
-  <gazebo reference="camera_lens">
-    <sensor type="camera" name="camera1">
-      <update_rate>30.0</update_rate>
-      <camera name="head">
-        <horizontal_fov>1.3962634</horizontal_fov>
-        <image>
-          <width>800</width>
-          <height>800</height>
-          <format>R8G8B8</format>
-        </image>
-        <clip>
-          <near>0.02</near>
-          <far>300</far>
-        </clip>
-        <noise>
-          <type>gaussian</type>
-          <!-- Noise is sampled independently per pixel on each frame.
-               That pixel's noise value is added to each of its color
-               channels, which at that point lie in the range [0,1]. -->
-          <mean>0.0</mean>
-          <stddev>0.007</stddev>
-        </noise>
-      </camera>
-      <plugin name="camera_controller" filename="libgazebo_ros_camera.so">
-        <alwaysOn>true</alwaysOn>
-        <updateRate>0.0</updateRate>
-        <cameraName>camera1</cameraName>
-        <imageTopicName>image_raw</imageTopicName>
-        <cameraInfoTopicName>camera_info</cameraInfoTopicName>
-        <frameName>camera_lens</frameName>
-        <hackBaseline>0.07</hackBaseline>
-        <distortionK1>0.0</distortionK1>
-        <distortionK2>0.0</distortionK2>
-        <distortionK3>0.0</distortionK3>
-        <distortionT1>0.0</distortionT1>
-        <distortionT2>0.0</distortionT2>
-      </plugin>
-    </sensor>
-  </gazebo>
-  <!--Camera  -->
+  <!-- ************************************ -->
+  <!-- ****** camera ****** -->
   <xacro:include filename="$(find farscope_group_proj)/urdf/simple_camera.urdf.xacro" />
   <!-- ************************************ -->
@@ -192,8 +151,11 @@
     <child link = "mpo_700_base_link" />
   </joint>
+  <xacro:arg name="camera_parent_link" default="forearm_link" />
+  <xacro:arg name="camera_origin_xyz" default="0 -0.08 0.38" />
+  <xacro:arg name="camera_origin_rpy" default="0 -1.5706 0" />
   <joint name="camera_to_robot" type="fixed">
-    <parent link="forearm_link" />
+    <parent link="$(arg camera_parent_link)" />
     <child link = "camera_link" />
-    <origin xyz="0 -0.08 0.38" rpy="0 -1.5706 0" />
+    <origin xyz="$(arg camera_origin_xyz)" rpy="$(arg camera_origin_rpy)" />
   </joint>
 </robot>

File: urdf/simple_camera.urdf.xacro (robot description, xacro)
@@ -59,3 +59,43 @@
     <origin xyz="0.03 0 0" rpy="0 0 0"/>
   </joint>
+  <!-- camera gazebo stuff -->
+  <gazebo reference="camera_lens">
+    <sensor type="camera" name="camera1">
+      <update_rate>30.0</update_rate>
+      <camera name="head">
+        <horizontal_fov>1.3962634</horizontal_fov>
+        <image>
+          <width>800</width>
+          <height>800</height>
+          <format>R8G8B8</format>
+        </image>
+        <clip>
+          <near>0.02</near>
+          <far>300</far>
+        </clip>
+        <noise>
+          <type>gaussian</type>
+          <!-- Noise is sampled independently per pixel on each frame.
+               That pixel's noise value is added to each of its color
+               channels, which at that point lie in the range [0,1]. -->
+          <mean>0.0</mean>
+          <stddev>0.007</stddev>
+        </noise>
+      </camera>
+      <plugin name="camera_controller" filename="libgazebo_ros_camera.so">
+        <alwaysOn>true</alwaysOn>
+        <updateRate>0.0</updateRate>
+        <cameraName>camera1</cameraName>
+        <imageTopicName>image_raw</imageTopicName>
+        <cameraInfoTopicName>camera_info</cameraInfoTopicName>
+        <frameName>camera_lens</frameName>
+        <hackBaseline>0.07</hackBaseline>
+        <distortionK1>0.0</distortionK1>
+        <distortionK2>0.0</distortionK2>
+        <distortionK3>0.0</distortionK3>
+        <distortionT1>0.0</distortionT1>
+        <distortionT2>0.0</distortionT2>
+      </plugin>
+    </sensor>
+  </gazebo>
 </robot>

Commit message: Adding cones, both using launch or world.

File: urdf/farscope_robot.urdf.xacro (robot description, xacro)
@@ -150,4 +150,5 @@
     <parent link="dummy_base" />
     <child link = "mpo_700_base_link" />
+    <origin xyz="0.0 0.0 0.0" rpy="0.0 0.0 0.0" />
   </joint>
   <xacro:arg name="camera_parent_link" default="forearm_link" />
