Commit message: Camera migrated to macro.  All works OK for visualizing.  TODO check the Gazebo end still works as well.

File: models/camera/simple_camera.urdf.xacro (robot description, xacro)
@@ -1,101 +1,108 @@
 <?xml version="1.0"?>
 <robot name="simple_camera" xmlns:xacro="http://ros.org/wiki/xacro">
-  <xacro:property name="camera_size" value="0.05" />
-  <link name="camera_link">
-    <collision>
-      <origin xyz="0 0 0" rpy="0 0 0"/>
-      <geometry>
-    <box size="${camera_size} ${camera_size} ${camera_size}"/>
-      </geometry>
-    </collision>
-    <visual>
-      <origin xyz="0 0 0" rpy="0 0 0"/>
-      <geometry>
-    <box size="${camera_size} ${camera_size} ${camera_size}"/>
-      </geometry>
-      <material name="cam_body">
-        <color rgba="0.7 0.7 0.8 1" />
-      </material>
-    </visual>
-    <inertial>
-      <mass value="1e-5" />
-      <origin xyz="0 0 0" rpy="0 0 0"/>
-      <inertia ixx="1e-6" ixy="0" ixz="0" iyy="1e-6" iyz="0" izz="1e-6" />
-    </inertial>
-  </link>
-  <gazebo reference="camera_link">
-    <material>Gazebo/Turquoise</material>
-  </gazebo>
-  <link name="camera_lens">
-    <collision>
-      <origin xyz="0.0 0.0 0.0" rpy="0.0 1.5706 0.0" />
-      <geometry>
-        <cylinder radius="0.02" length="0.01" />
-      </geometry>
-    </collision>
-    <visual>
-      <origin xyz="0.0 0.0 0.0" rpy="0.0 1.5706 0.0" />
-      <origin xyz="0 0 0" rpy="0 0 0"/>
-      <geometry>
-        <cylinder radius="0.02" length="0.01" />
-      </geometry>
-      <material name="cam_lens">
-        <color rgba="0.1 0.1 0.1 1" />
-      </material>
-    </visual>
-    <inertial>
-      <mass value="1e-5" />
-      <origin xyz="0.0 0.0 0.0" rpy="0.0 1.5706 0.0" />
-      <origin xyz="0 0 0" rpy="0 0 0"/>
-      <inertia ixx="1e-6" ixy="0" ixz="0" iyy="1e-6" iyz="0" izz="1e-6" />
-    </inertial>
-  </link>
-  <gazebo reference="camera_lens">
-    <material>Gazebo/DarkGrey</material>
-  </gazebo>
-  <joint name="camera_to_lens" type="fixed">
-    <parent link="camera_link" />
-    <child link = "camera_lens" />
-    <origin xyz="0.03 0 0" rpy="0 0 0"/>
-  </joint>
-  <!-- camera gazebo stuff -->
-  <gazebo reference="camera_lens">
-    <sensor type="camera" name="camera1">
-      <update_rate>30.0</update_rate>
-      <camera name="head">
-        <horizontal_fov>1.3962634</horizontal_fov>
-        <image>
-          <width>800</width>
-          <height>800</height>
-          <format>R8G8B8</format>
-        </image>
-        <clip>
-          <near>0.02</near>
-          <far>300</far>
-        </clip>
-        <noise>
-          <type>gaussian</type>
-          <!-- Noise is sampled independently per pixel on each frame.
-               That pixel's noise value is added to each of its color
-               channels, which at that point lie in the range [0,1]. -->
-          <mean>0.0</mean>
-          <stddev>0.007</stddev>
-        </noise>
-      </camera>
-      <plugin name="camera_controller" filename="libgazebo_ros_camera.so">
-        <alwaysOn>true</alwaysOn>
-        <updateRate>0.0</updateRate>
-        <cameraName>camera1</cameraName>
-        <imageTopicName>image_raw</imageTopicName>
-        <cameraInfoTopicName>camera_info</cameraInfoTopicName>
-        <frameName>camera_lens</frameName>
-        <hackBaseline>0.07</hackBaseline>
-        <distortionK1>0.0</distortionK1>
-        <distortionK2>0.0</distortionK2>
-        <distortionK3>0.0</distortionK3>
-        <distortionT1>0.0</distortionT1>
-        <distortionT2>0.0</distortionT2>
-      </plugin>
-    </sensor>
-  </gazebo>
+  <xacro:macro name="simple_camera" params="camera_name parent_link *origin">
+    <xacro:property name="camera_size" value="0.05" />
+    <link name="${camera_name}_link">
+      <collision>
+        <origin xyz="0 0 0" rpy="0 0 0"/>
+        <geometry>
+      <box size="${camera_size} ${camera_size} ${camera_size}"/>
+        </geometry>
+      </collision>
+      <visual>
+        <origin xyz="0 0 0" rpy="0 0 0"/>
+        <geometry>
+      <box size="${camera_size} ${camera_size} ${camera_size}"/>
+        </geometry>
+        <material name="cam_body">
+          <color rgba="0.7 0.7 0.8 1" />
+        </material>
+      </visual>
+      <inertial>
+        <mass value="1e-5" />
+        <origin xyz="0 0 0" rpy="0 0 0"/>
+        <inertia ixx="1e-6" ixy="0" ixz="0" iyy="1e-6" iyz="0" izz="1e-6" />
+      </inertial>
+    </link>
+    <gazebo reference="${camera_name}_link">
+      <material>Gazebo/Turquoise</material>
+    </gazebo>
+    <link name="${camera_name}_lens">
+      <collision>
+        <origin xyz="0.0 0.0 0.0" rpy="0.0 1.5706 0.0" />
+        <geometry>
+          <cylinder radius="0.02" length="0.01" />
+        </geometry>
+      </collision>
+      <visual>
+        <origin xyz="0.0 0.0 0.0" rpy="0.0 1.5706 0.0" />
+        <origin xyz="0 0 0" rpy="0 0 0"/>
+        <geometry>
+          <cylinder radius="0.02" length="0.01" />
+        </geometry>
+        <material name="cam_lens">
+          <color rgba="0.1 0.1 0.1 1" />
+        </material>
+      </visual>
+      <inertial>
+        <mass value="1e-5" />
+        <origin xyz="0.0 0.0 0.0" rpy="0.0 1.5706 0.0" />
+        <origin xyz="0 0 0" rpy="0 0 0"/>
+        <inertia ixx="1e-6" ixy="0" ixz="0" iyy="1e-6" iyz="0" izz="1e-6" />
+      </inertial>
+    </link>
+    <gazebo reference="${camera_name}_lens">
+      <material>Gazebo/DarkGrey</material>
+    </gazebo>
+    <joint name="${camera_name}_to_lens" type="fixed">
+      <parent link="${camera_name}_link" />
+      <child link = "${camera_name}_lens" />
+      <origin xyz="0.03 0 0" rpy="0 0 0"/>
+    </joint>
+    <joint name="${camera_name}_to_parent" type="fixed">
+      <parent link="${parent_link}" />
+      <child link = "${camera_name}_link" />
+      <xacro:insert_block name="origin" />
+    </joint>
+    <!-- camera gazebo stuff -->
+    <gazebo reference="${camera_name}_lens">
+      <sensor type="camera" name="${camera_name}">
+        <update_rate>30.0</update_rate>
+        <camera name="${camera_name}_cam">
+          <horizontal_fov>1.3962634</horizontal_fov>
+          <image>
+            <width>800</width>
+            <height>800</height>
+            <format>R8G8B8</format>
+          </image>
+          <clip>
+            <near>0.02</near>
+            <far>300</far>
+          </clip>
+          <noise>
+            <type>gaussian</type>
+            <!-- Noise is sampled independently per pixel on each frame.
+                That pixel's noise value is added to each of its color
+                channels, which at that point lie in the range [0,1]. -->
+            <mean>0.0</mean>
+            <stddev>0.007</stddev>
+          </noise>
+        </camera>
+        <plugin name="camera_controller" filename="libgazebo_ros_camera.so">
+          <alwaysOn>true</alwaysOn>
+          <updateRate>0.0</updateRate>
+          <cameraName>${camera_name}</cameraName>
+          <imageTopicName>image_raw</imageTopicName>
+          <cameraInfoTopicName>camera_info</cameraInfoTopicName>
+          <frameName>${camera_name}_lens</frameName>
+          <hackBaseline>0.07</hackBaseline>
+          <distortionK1>0.0</distortionK1>
+          <distortionK2>0.0</distortionK2>
+          <distortionK3>0.0</distortionK3>
+          <distortionT1>0.0</distortionT1>
+          <distortionT2>0.0</distortionT2>
+        </plugin>
+      </sensor>
+    </gazebo>
+  </xacro:macro>
 </robot>

File: models/example_robot/farscope_example_robot.urdf.xacro (robot description, xacro)
@@ -9,14 +9,11 @@
     <origin xyz="0.0 0.0 0.0" rpy="0.0 0.0 0.0" />
   </xacro:simple_gripper>
-  <!-- ************************************ -->
-  <!-- ****** camera ****** -->
+  <!-- ****** cameras ****** -->
   <xacro:include filename="$(find farscope_group_proj)/models/camera/simple_camera.urdf.xacro" />
-  <xacro:arg name="camera_parent_link" default="forearm_link" />
-  <xacro:arg name="camera_origin_xyz" default="0 -0.08 0.38" />
-  <xacro:arg name="camera_origin_rpy" default="0 -1.5706 0" />
-  <joint name="camera_to_robot" type="fixed">
-    <parent link="$(arg camera_parent_link)" />
-    <child link = "camera_link" />
-    <origin xyz="$(arg camera_origin_xyz)" rpy="$(arg camera_origin_rpy)" />
-  </joint>
+  <xacro:simple_camera camera_name="camera1" parent_link="forearm_link" >
+    <origin xyz="0 -0.08 0.38" rpy="0 -1.5706 0" />
+  </xacro:simple_camera>
+  <xacro:simple_camera camera_name="camera2" parent_link="upper_arm_link" >
+    <origin xyz="0 0 0.7" rpy="0 -0.75 0" />
+  </xacro:simple_camera>
 </robot>
