Commit message: All working in Gazebo again and with tidier file arrangements.  TODO randomness in the target spawning.

File: models/target/target.urdf (robot description, URDF)
Before this commit: robot farscope_target, 1 links, 0 joints
Links:
- link link_0: geometry collision mesh filename=package://farscope_group_proj/models/target/target.stl; visual mesh filename=package://farscope_group_proj/models/target/target.stl
