Commit message: Now mobile arm implemented as xacro macro.

File: models/example_robot/farscope_example_robot.urdf.xacro (robot description, xacro)
@@ -2,6 +2,6 @@
 <robot name="farscope_example_robot" xmlns:xacro="http://ros.org/wiki/xacro">
   <!-- mobile base -->
-  <xacro:include filename="$(find farscope_group_proj)/models/robot_base/mobile_manipulator.urdf.xacro" />
-  <xacro:mobile_manipulator />
+  <xacro:include filename="$(find farscope_group_proj)/models/mobile_arm/mobile_arm.urdf.xacro" />
+  <xacro:mobile_arm />
   <!-- ****** gripper ****** -->
   <xacro:include filename="$(find farscope_group_proj)/models/gripper/simple_gripper.urdf.xacro" />
@@ -10,145 +10,6 @@
   </xacro:simple_gripper>
   <!-- ************************************ -->
-  <!-- ****** arm stuff ****** -->
-  <!-- copied from ur_description/urdf/ur10_joint_limited.urdf.xacro -->
-  <!-- common stuff -->
-  <xacro:include filename="$(find ur_description)/urdf/common.gazebo.xacro" />
-  <!-- ur10 macro -->
-  <xacro:include filename="$(find ur_description)/urdf/ur10.urdf.xacro" />
-  <!-- make the arm -->
-  <xacro:ur10_robot prefix="" joint_limited="true"
-    shoulder_pan_lower_limit="${-pi}" shoulder_pan_upper_limit="${pi}"
-    shoulder_lift_lower_limit="${-pi}" shoulder_lift_upper_limit="${pi}"
-    elbow_joint_lower_limit="${-pi}" elbow_joint_upper_limit="${pi}"
-    wrist_1_lower_limit="${-pi}" wrist_1_upper_limit="${pi}"
-    wrist_2_lower_limit="${-pi}" wrist_2_upper_limit="${pi}"
-    wrist_3_lower_limit="${-pi}" wrist_3_upper_limit="${pi}"
-    transmission_hw_interface="hardware_interface/PositionJointInterface"
-/>
-  <!-- ************************************ -->
-  <!-- ****** build the mobile base ****** -->
-  <!-- adapting from neo_simulation:mmo700.urdf.xacro -->
-  <!--mmo700 common stuff SKIPPED because it reloads controllers and grasp fix-->
-  <!-- <xacro:include filename="$(find neo_simulation)/robots/mmo_700/urdf/xacros/common.gazebo.xacro" /> -->
-  <!-- CABINET -->
-  <xacro:include filename="$(find neo_simulation)/robots/mmo_700/urdf/xacros/cabinet.xacro" />
-  <!-- Body -->
-  <xacro:include filename="$(find neo_simulation)/robots/mmo_700/urdf/xacros/mpo_700_body.xacro" />
-  <!-- SENSORS -->
-  <!-- Sick-S300 -->
-  <!-- <xacro:include filename="$(find neo_simulation)/robots/mmo_700/xacros/sick_S300.xacro" /> -->
-  <!--Sick Micro-scan  -->
-  <xacro:include filename="$(find neo_simulation)/robots/mmo_700/urdf/xacros/micro_scan.xacro" />
-  <!-- Gazebo -->
-  <!-- <xacro:include filename="$(find neo_simulation)/robots/mmo_700/urdf/xacros/mpo_700_gazebo.xacro" /> -->
-  <!-- copied from mpo_700_gazebo.xacro -->
-  <gazebo reference="mpo_700_base_link">
-    <gravity>true</gravity>
-    <self_collide>false</self_collide>
-  </gazebo>
-  <gazebo>
-    <plugin name="mpo_700_controller" filename="libgazebo_ros_planar_move.so">
-        <commandTopic>cmd_vel</commandTopic>
-        <odometryTopic>odom</odometryTopic>
-        <odometryFrame>odom</odometryFrame>
-        <odometryRate>20.0</odometryRate>
-        <robotBaseFrame>mpo_700_base_link</robotBaseFrame>
-    </plugin>
-  </gazebo>
-  <!-- Head -->
-  <xacro:include filename="$(find neo_simulation)/robots/mmo_700/urdf/xacros/mpo_700_caster.xacro" />
-  <!-- Wheel -->
-  <xacro:include filename="$(find neo_simulation)/robots/mmo_700/urdf/xacros/mpo_700_wheel.xacro" />
-  <!-- Base Macro-->
-  <xacro:mpo_700_base name="mpo_700_base_link">
-  </xacro:mpo_700_base>
-  <!-- Casters -->
-  <xacro:mpo_700_caster_0 name="mpo_700_caster_front_left" parent="mpo_700_base_link">
-    <origin xyz="0.24 0.18 0.27" rpy="3.14 0 -1.57" />
-  </xacro:mpo_700_caster_0>
-  <xacro:mpo_700_caster_1 name="mpo_700_caster_front_right" parent="mpo_700_base_link">
-    <origin xyz="0.24 -0.18 0.27" rpy="3.14 0 1.57" />
-  </xacro:mpo_700_caster_1>
-  <xacro:mpo_700_caster_2 name="mpo_700_caster_back_left" parent="mpo_700_base_link">
-    <origin xyz="-0.24 0.18 0.27" rpy="3.14 0 -1.57" />
-  </xacro:mpo_700_caster_2>
-  <xacro:mpo_700_caster_3 name="mpo_700_caster_back_right" parent="mpo_700_base_link">
-    <origin xyz="-0.24 -0.18 0.27" rpy="3.14 0 1.57" />
-  </xacro:mpo_700_caster_3>
-  <!-- wheels -->
-  <xacro:mpo_700_wheel name="mpo_700_wheel_front_left" parent="mpo_700_caster_front_left_link">
-    <origin xyz="-0.05 0. 0.18" rpy="0 0 0" />
-  </xacro:mpo_700_wheel>
-  <xacro:mpo_700_wheel name="mpo_700_wheel_front_right" parent="mpo_700_caster_front_right_link">
-    <origin xyz="-0.05 0. 0.18" rpy="0 0 0" />
-  </xacro:mpo_700_wheel>
-  <xacro:mpo_700_wheel name="mpo_700_wheel_back_left" parent="mpo_700_caster_back_left_link">
-    <origin xyz="-0.05 0. 0.18" rpy="0 0 0" />
-  </xacro:mpo_700_wheel>
-  <xacro:mpo_700_wheel name="mpo_700_wheel_back_right" parent="mpo_700_caster_back_right_link">
-    <origin xyz="-0.05 0. 0.18" rpy="0 0 0" />
-  </xacro:mpo_700_wheel>
-  <!--cabinet-->
-  <xacro:mmo_700_cabinet name="cabinet" parent="mpo_700_base_link">
-  	<origin xyz="0.072 0 0.35" rpy="0 0 0" />
-  </xacro:mmo_700_cabinet>
-  <!-- LIDAR -->
-  <xacro:sick_laser_v0 name="lidar_1" parent="mpo_700_base_link" ros_topic="lidar_1/scan_filtered">
-  <origin xyz="0.360 0 0.181" rpy="3.14 0 0" />
-  </xacro:sick_laser_v0>
-  <!-- Lidar sensors -->
-  <gazebo reference="lidar_1_link">
-      <sensor type="ray" name="lidar_1_sensor">
-          <pose>0 0 0 0 0 0</pose>
-          <visualize>false</visualize>
-          <update_rate>40</update_rate>
-          <ray>
-            <scan>
-              <horizontal>
-                <samples>720</samples>
-                <resolution>1</resolution>
-                <min_angle>-1.48</min_angle>
-                <max_angle>1.48</max_angle>
-              </horizontal>
-            </scan>
-            <range>
-              <min>0.10</min>
-              <max>30.0</max>
-              <resolution>0.05</resolution>
-            </range>
-            <noise>
-              <type>gaussian</type>
-              <!-- Noise parameters based on published spec for Hokuyo laser
-                   achieving "+-30mm" accuracy at range < 10m.  A mean of 0.0m and
-                   stddev of 0.01m will put 99.7% of samples within 0.03m of the true
-                   reading. -->
-              <mean>0.0</mean>
-              <stddev>0.01</stddev>
-            </noise>
-          </ray>
-          <plugin name="lidar_1" filename="libgazebo_ros_laser.so">
-            <topicName>lidar_1/scan_filtered</topicName>
-            <frameName>lidar_1_link</frameName>
-          </plugin>
-        </sensor>
-  </gazebo>
-  <!-- ************************************ -->
   <!-- ****** camera ****** -->
   <xacro:include filename="$(find farscope_group_proj)/models/camera/simple_camera.urdf.xacro" />
-  <!-- ************************************ -->
-  <!-- ****** integration ****** -->
-  <!-- fix the arm to the cabinet -->
-  <joint name="arm_to_cabinet" type="fixed">
-    <parent link="cabinet_link" />
-    <child link = "base_link" />
-    <origin xyz="0.133 0.0 0.416" rpy="0.0 0.0 0.0" />
-  </joint>
-  <!-- dummy link to avoid inertia warning -->
-  <link name="dummy_base" />
-  <joint name="dummy_joint" type="fixed">
-    <parent link="dummy_base" />
-    <child link = "mpo_700_base_link" />
-    <origin xyz="0.0 0.0 0.0" rpy="0.0 0.0 0.0" />
-  </joint>
   <xacro:arg name="camera_parent_link" default="forearm_link" />
   <xacro:arg name="camera_origin_xyz" default="0 -0.08 0.38" />

Commit message: Fixing naming issues - all to farscope_group_project

File: models/example_robot/farscope_example_robot.urdf.xacro (robot description, xacro)
@@ -2,13 +2,13 @@
 <robot name="farscope_example_robot" xmlns:xacro="http://ros.org/wiki/xacro">
   <!-- mobile base -->
-  <xacro:include filename="$(find farscope_group_proj)/models/mobile_arm/mobile_arm.urdf.xacro" />
+  <xacro:include filename="$(find farscope_group_project)/models/mobile_arm/mobile_arm.urdf.xacro" />
   <xacro:mobile_arm />
   <!-- ****** gripper ****** -->
-  <xacro:include filename="$(find farscope_group_proj)/models/gripper/simple_gripper.urdf.xacro" />
+  <xacro:include filename="$(find farscope_group_project)/models/gripper/simple_gripper.urdf.xacro" />
   <xacro:simple_gripper parent_link="tool0">
     <origin xyz="0.0 0.0 0.0" rpy="0.0 0.0 0.0" />
   </xacro:simple_gripper>
   <!-- ****** cameras ****** -->
-  <xacro:include filename="$(find farscope_group_proj)/models/camera/simple_camera.urdf.xacro" />
+  <xacro:include filename="$(find farscope_group_project)/models/camera/simple_camera.urdf.xacro" />
   <xacro:simple_camera camera_name="camera1" parent_link="forearm_link" >
     <origin xyz="0 -0.08 0.38" rpy="0 -1.5706 0" />

File: models/target/target.urdf (robot description, URDF)
Before this commit: robot farscope_target, 1 links, 0 joints
Links:
- link link_0: geometry collision mesh filename=package://farscope_group_project/models/target/target.stl; visual mesh filename=package://farscope_group_project/models/target/target.stl
